File: adc/kicad/adc.kicad_sch (KiCad schematic)
At the start: 68 parts, among them J1 Conn_01x02_Pin, J2 Conn_01x04_Pin, J3 Conn_01x02_Pin, J4 Conn_01x02_Pin, J5 pcie_98, U2 ESD5344D-TP, U3 ADS1261B, U4 ESD5344D-TP, U5 TPS7A2050PDBVR, U6 TPS61252DSG, U7 XC6206P332MR

Commit message: Progressing on the ADC card schematic.
Parts:
- removed C17, C18, C19, C21: 10u, Capacitor_SMD:C_0603_1608Metric, symbol Device:C_Small
- removed C20, C22: 100n, Capacitor_SMD:C_0402_1005Metric, symbol Device:C_Small
- removed FB1: Ferrite Bead, Inductor_SMD:L_0805_2012Metric, symbol Device:FerriteBead_Small
- removed J3, J4: Conn_01x02_Pin, symbol Connector:Conn_01x02_Pin
- removed L1: 1uH, Inductor_SMD:L_1210_3225Metric, symbol Device:L_Iron
- removed R28: 22K, Resistor_SMD:R_0402_1005Metric, symbol Device:R_Small_US
- removed U2: ESD5344D-TP, common:Diodes_UDFN-10_1.0x2.5mm_P0.5mm, symbol common:ESD5344D
- removed U5: TPS7A2050PDBVR, adc:SOT-23-5, symbol adc:TPS7A2050
- removed U6: TPS61252DSG, adc:WSON-8-1EP_2x2mm_P0.5mm_EP0.9x1.6mm, symbol adc:TPS61252DSG
- added C1, C2, C3: ~, Capacitor_SMD:C_0402_1005Metric, symbol Device:C_Small
- added C14: 33n, Capacitor_SMD:C_0402_1005Metric, symbol Device:C_Small
- added C15: 330n, Capacitor_SMD:C_0402_1005Metric, symbol Device:C_Small
- added C25, C27, C34, C36, C38, C39: 100n, Capacitor_SMD:C_0402_1005Metric, symbol Device:C_Small
- added C26, C28, C37, C40: 10u, Capacitor_SMD:C_0603_1608Metric, symbol Device:C_Small
- added C33, C41, C42: 10u, symbol Device:C_Small
- added C4: 2u2, Capacitor_SMD:C_0402_1005Metric, symbol Device:C_Small
- added C43: 100n, symbol Device:C_Small
- added D2, D3, D4, D5: RED, LED_SMD:LED_0603_1608Metric, symbol Device:LED
- added J1, J2: Conn_01x02_Pin, symbol Connector:Conn_01x02_Pin
- added L1: 2u2H, Inductor_SMD:L_0805_2012Metric, symbol Device:L_Ferrite
- added R13, R14, R17: 2K, Resistor_SMD:R_0402_1005Metric, symbol Device:R_Small_US
- added R31: 360K, Resistor_SMD:R_0402_1005Metric, symbol Device:R_Small_US
- added R32: 100K, Resistor_SMD:R_0402_1005Metric, symbol Device:R_Small_US
- added R33: 464K, Resistor_SMD:R_0402_1005Metric, symbol Device:R_Small_US
- added R5, R8: ~, Resistor_SMD:R_0402_1005Metric, symbol Device:R_Small_US
- added U3: TPS7A2050PDBVR, adc:SOT-23-5, symbol adc:TPS7A2050
- added U4: TPS7A2025PDBVR, adc:SOT-23-5, symbol adc:TPS7A2050
- added U6: TPS65135, symbol adc:TPS65135
- added U7: ADP7182AUJZ-5.0, Package_TO_SOT_SMD:TSOT-23-5, symbol Regulator_Linear:ADP7182AUJZ-5.0
- added U8: ADP7182AUJZ-2.5, Package_TO_SOT_SMD:TSOT-23-5, symbol Regulator_Linear:ADP7182AUJZ-2.5
- C10: renamed from C1; LCSC C52923 -> (none)
- C11: renamed from C2; LCSC C52923 -> (none)
- C12: renamed from C3; LCSC C1525 -> (none)
- C13: renamed from C4; LCSC C1525 -> (none)
- C16: value 100pf -> 33n; LCSC C1546 -> (none)
- C17: renamed from C12; LCSC C1538 -> (none)
- C21: renamed from C14; LCSC C52923 -> (none)
- C22: renamed from C15; LCSC C96446 -> (none)
- C23, C24: value 10u -> 100n; footprint Capacitor_SMD:C_0603_1608Metric -> Capacitor_SMD:C_0402_1005Metric; LCSC C96446 -> (none)
- C29: renamed from C25; LCSC C96446 -> (none)
- C30: renamed from C26; LCSC C1525 -> (none)
- C31: renamed from C27; LCSC C1525 -> (none)
- C32: renamed from C28; LCSC C96446 -> (none)
- C5: value 1u -> 2u2; LCSC C52923 -> (none)
- C6: LCSC C1523 -> (none)
- C7, C8: value 2u2 -> ~; LCSC C1523 -> (none)
- C9: value 1u -> ~; LCSC C52923 -> (none)
- D1: footprint LED_SMD:LED_0805_2012Metric -> LED_SMD:LED_0603_1608Metric; LCSC C84256 -> C2286
- R1, R2: value 51K -> 1K 0.1%; LCSC C25794 -> (none)
- R10, R12: value 10K -> 1K 0.1%
- R11: value 2K2 0.1% -> 1K 0.1%
- R15: renamed from R5; LCSC C25794 -> (none)
- R16: renamed from R6; LCSC C25794 -> (none)
- R18: renamed from R15; LCSC C25118 -> (none)
- R19: renamed from R16; LCSC C25118 -> (none)
- R20: renamed from R14; value 100R -> 510R; LCSC C25076 -> (none)
- R21: renamed from R17; LCSC C25118 -> (none)
- R22: renamed from R18; LCSC C25118 -> (none)
- R23: value 510K -> 5K1; LCSC C11616 -> (none)
- R24: LCSC C25905 -> (none)
- R25: value 120K -> 5K1; LCSC C25750 -> (none)
- R26: value 20K -> 5K1; LCSC C25765 -> (none)
- R27: value 0R -> 5K1; footprint Resistor_SMD:R_0805_2012Metric -> Resistor_SMD:R_0402_1005Metric; LCSC C17477 -> (none)
- R28: renamed from R22; LCSC C25794 -> (none)
- R29: renamed from R21; LCSC C25794 -> (none)
- R3: renamed from R8; value 2K2 0.1% -> 1K 0.1%
- R30: renamed from R19; value 100R -> 510R; LCSC C25076 -> (none)
- R4, R7: value 51K -> ~; LCSC C25794 -> (none)
- R6: renamed from R3; value 10K -> ~
- R9: value 2K2 0.1% -> ~
- U1: renamed from U3; LCSC DNP -> (none)
- U2: renamed from U4; LCSC C2841840 -> (none)
- U5: renamed from U7; LCSC C5446 -> (none)
- renumbered C10 to C18, C11 to C19, C13 to C20, J1 to J3, J5 to J4, J2 to J5
Connections:
- net +5VA: now also R23.1, C25.2, C26.2, R13.2, U3.5 (OUT), U4.1 (IN), U4.3 (EN); no longer C10.2, C12.2, C23.2, R1.2, R11.2, R3.2, R4.2, R9.2, U1.4 (AVDD)
- net +5VD: now also C42.1, U6.1 (VIN)
- net AIN0: now also C14.1, C15.1, R13.1, R14.2; no longer C19.2, C20.2, R30.2
- net AIN1: now also C16.2, C15.2, R14.1, R17.1; no longer C18.1, C19.1, R20.2
- net AIN2: now also C18.1, C19.1, R20.2; no longer R6.2
- net AIN3: now also C19.2, C20.2, R30.2; no longer R10.2
- net AIN4: now also C6.1, R6.2, C3.2; no longer R12.2
- net GNDA: now also C16.1, C9.2, D1.1 (K), U1.1 (AINCOM), C1.1, C14.2, C2.1, C25.1, C26.1, C27.1, C28.1, C3.1, C33.2, C34.1, C36.1, C37.1, C38.1, C39.1, C40.1, C41.1, C42.2, C43.2, D2.1 (K), D3.1 (K), D4.1 (K), D5.1 (K), U3.2 (GND), U4.2 (GND), U6.11 (PGND), U6.12 (PGND), U6.5 (GND), U7.1 (GND), U8.1 (GND); no longer C5.1, C6.2, C9.1, J3.1 (Pin_1), J5.1 (Pin_1), R2.1, R27.2, R7.1, U1.33 (AVSS), U1.5 (AVSS)
- net GNDD: no longer D1.1 (K), R26.2, R27.1
- net -2V5A: now reaches R11.1, R12.1
- net -2V5A: now also R10.1, R26.1, U1.33 (AVSS), U1.5 (AVSS), C39.2, C40.2, U8.5 (VOUT); no longer C8.1
- net at J3.2 (Pin_2), R3.1, R6.1: no longer C6.1
- net +2V5A: now reaches R25.1
- net +2V5A: now also C10.2, C12.2, R1.2, R2.2, R3.2, U1.4 (AVDD), C27.2, C28.2, U4.5 (OUT)
- net at D1.2 (A): now also R23.2; no longer R24.2
- net +3V3 renamed +3V3D
- net +3V3D: now also R27.1
- new net: J3.1 (Pin_1), R12.2, R9.1
- new net: D4.2 (A), R26.2
- new net: R31.2, R32.1, U6.7 (FB)
- new net: D3.2 (A), R25.2
- new net: J1.2 (Pin_2), R1.1, R4.1
- new net: R32.2, R33.1, U6.6 (FBG)
- new net: J2.1 (Pin_1), R11.2, R8.1
- new net: D2.2 (A), R24.2
- new net: J1.1 (Pin_1), R10.2, R7.1
- new net: J2.2 (Pin_2), R2.1, R5.1
- new net: L1.2, U6.13 (L2), U6.14 (L2)
- new net: L1.1, U6.15 (L1), U6.16 (L1)
- new net: C43.1, U6.4 (VAUX)
- new net: D5.2 (A), R27.2
- new net +5V7: C23.2, C33.1, R31.1, U3.1 (IN), U3.3 (EN), U6.10 (OUTP), U6.9 (OUTP)
- new net -5V7: C34.2, C41.2, R33.2, U6.2 (OUTN), U6.3 (OUT2), U7.2 (VIN), U7.3 (EN)
- new net -5VA: C36.2, C37.2, C38.2, J5.1 (Pin_1), R17.2, R24.1, U7.5 (VOUT), U8.2 (VIN), U8.3 (EN)
- new net AIN5: C6.2, C9.1, R9.2, U1.27 (AIN5)
- new net AIN6: C1.2, C4.1, R4.2, U1.26 (AIN6)
- new net AIN7: C4.2, C7.1, R7.2, U1.25 (AIN7)
- new net AIN8: C2.2, C5.1, R5.2, U1.24 (AIN8)
- new net AIN9: C5.2, C8.1, R8.2, U1.23 (AIN9)
- no-connect marks 9 -> 7
Other:
- note added: "Have long pads for SMD footprints, for hand soldering."
- note added: "LOAD CELL INPUT AND REFERENCE"
- note removed: "5.77V NOMINAL"
- note removed: "ANALOG 5V"
- note removed: "Consider thermistor circuit from the ADS1120 datasheet."
- note removed: "Consider to run the thermistors on 3.3 volt to reduce power disspation."
- note removed: "LOAD CELL"
- note removed: "NOTE: AINCOM users its own voltage divider to simplify two layers PCB layout."
- note removed: "NOTE: All sensor measurements are ratiometric, proportional to (5VA - GNDA)."
- note removed: "TODO: Add jumpers for two SPI channels."
- note removed: "TODO: Consider to add constant current NTC 50K thermistor inputs."
- note removed: "TODO: Should MOSI be pulled up or down?"
- moved on the sheet: C10, C11, C12, C13, C17, C18, C19, C20, C21, C22, C29, C30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

Commit message: Progress with the ADC's schematic.
Parts:
- removed J4: pcie_98, common:PCIE_98_CARD, symbol common:PCIE_98_EDGE
- removed U5: XC6206P332MR, Package_TO_SOT_SMD:SOT-23-3, symbol ble:HT75xx-1-SOT89
- added J6: pcie_98, common:PCIE_98_CARD, symbol common:PCIE_98_EDGE
- added R34: 470R, Resistor_SMD:R_0402_1005Metric, symbol Device:R_Small_US
- added R35, R36: 1K 0.1% 10ppm, Resistor_SMD:R_0402_1005Metric, symbol Device:R_Small_US
- added R37: 0R, Resistor_SMD:R_0805_2012Metric, symbol Device:R_Small_US
- added U9: XC6206P332MR, symbol breakout:XC6206P332MR
- C1: value ~ -> 2u2; LCSC (none) -> C12530
- C10, C11, C21: LCSC (none) -> C52923
- C12, C13, C23, C24, C25, C27, C30, C31, C34, C36, C38, C39: LCSC (none) -> C1525
- C14, C16, C18, C20: value 33n -> 47n; LCSC (none) -> C327054
- C15, C19: value 330n -> 470n; LCSC (none) -> C47339
- C17: LCSC (none) -> C1538
- C2, C3, C7, C8, C9: value ~ -> 100n; LCSC (none) -> C1525
- C22, C26, C28, C29, C32, C37, C40: LCSC (none) -> C19702
- C33, C41, C42: footprint (none) -> Capacitor_SMD:C_0603_1608Metric; LCSC (none) -> C19702
- C4: value 2u2 -> 100n; LCSC (none) -> C1525
- C43: footprint (none) -> Capacitor_SMD:C_0402_1005Metric; LCSC (none) -> C1525
- C5, C6: LCSC (none) -> C12530
- R1, R12, R2, R3: value 1K 0.1% -> 1K 0.1% 10ppm; LCSC (none) -> C328418
- R10, R11: value 1K 0.1% -> 470R; LCSC (none) -> C25117
- R13, R14, R17: value 2K -> 1K 0.1% 10ppm; LCSC (none) -> C328418
- R15, R16, R28, R29: LCSC (none) -> C25794
- R18, R19, R21, R22: LCSC (none) -> C25118
- R20: value 510R -> 470R; LCSC (none) -> C25117
- R23, R24, R25, R26, R27: LCSC (none) -> C25905
- R30: value 510R -> 1K 0.1% 10ppm; LCSC (none) -> C328418
- R31: value 360K -> 360K 0.1%; LCSC (none) -> C2759490
- R32: value 100K -> 100K 0.1%; LCSC (none) -> C852328
- R33: value 464K -> 464K 0.1%; LCSC (none) -> C172084
- R4, R5, R6, R9: value ~ -> 470R; LCSC (none) -> C25117
- R7, R8: value ~ -> 1K 0.1% 10ppm; LCSC (none) -> C328418
- U1, U3, U4, U7, U8: LCSC (none) -> DIGIKEY
- U2: LCSC (none) -> C2841840
- U6: LCSC (none) -> C57950
Connections:
- net +2V5A: now also R7.2; no longer R2.2
- net +3V3D: now also U9.2 (VOUT)
- net +5VA: now also R17.2; no longer R13.2
- net +5VD: now also U6.8 (EN), J6.B1 (Pin_b1), J6.B2 (Pin_b2), J6.B3 (Pin_b3), J6.B4 (Pin_b4), U9.3 (VIN)
- net -2V5A: now also R2.1, R8.1; no longer R10.1, R11.1
- net -5VA: now also R35.2; no longer R17.2
- net AIN1: now also R30.1, R36.1; no longer R14.1, R17.1
- net AIN2: now also R34.2; no longer R20.2
- net AIN3: now also R20.2; no longer R30.2
- net AIN6: now also C1.1, C2.2; no longer C1.2, C4.1
- net AIN7: now also C1.2, C4.1, R5.2; no longer C4.2, C7.1, R7.2
- net AIN8: now also C7.2, R10.2; no longer C2.2, R5.2
- net AIN9: now also R11.2; no longer R8.2
- net GNDA: now also C4.2, C7.1, R37.1; no longer C1.1, C7.2
- net GNDD: now also J6.A1 (Pin_a1), J6.A2 (Pin_a2), J6.A3 (Pin_a3), J6.A4 (Pin_a4), R37.2, U9.1 (GND)
- net PA5: now also J6.B28 (Pin_b28)
- net PA6: now also J6.B21 (Pin_b21)
- net PA7: now also J6.A27 (Pin_a27)
- net PB14: now also J6.B14 (Pin_b14)
- net at J5.2 (Pin_2): now also R20.1; no longer R30.1
- net at J5.3 (Pin_3): now also R34.1; no longer R20.1
- new net: J1.1 (Pin_1), R2.2, R5.1
- new net: R35.1, R36.2
- new net: R14.1, R30.2
- new net: J2.2 (Pin_2), R10.1, R7.1
- new net: J2.1 (Pin_1), R11.1, R8.2
- new net: R13.2, R17.1
- no-connect marks 7 -> 93
Other:
- note added: "(AIN2-AIN3)/(AIN0-AIN1)"
- note added: "(AIN4-AIN5)/(AVDD-AVSS)"
- note added: "(AIN6-AIN7)/(AVDD-AVSS)"
- note added: "(AIN8-AIN9)/(AVDD-AVSS)"
- note added: "Add to the load cell connector pin for ground/shield"
- note added: "Adjust the symbols of the positive and negative regulators to look the same."
- note added: "Consider to make the load cell connector 6 pins Kelvin style (with solder jumps for bypassing the Kelvin arrangment)"
- note added: "Do the negative regulators also have pin 4 NC?"
- note added: "LOAD CELL"
- note removed: "LOAD CELL INPUT AND REFERENCE"
- moved on the sheet: C29, C30, C31, C32, C33, C41, C42, C43, D1, D2, D3, D4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
