File: adc/kicad/sim/sim.kicad_sch (KiCad schematic)
At the start: 13 parts

Commit message: Progress with the ADC's schematic.
Parts:
- C1, C2: value 33n -> 47n
- C3: value 330n -> 470n
- R5, R6: value 100 -> 470
Connections:
- no-connect marks 0 -> 2
Other:
- note added: "ADC"
- note added: "LOAD CELL"
- moved on the sheet: C1, C2, C3, MES1, R5, R6, R7

Commit message: Updated RC values in the loadcell simulation.
Parts:
- C1, C2: value 47n -> 22n
- C3: value 470n -> 220n
- R5, R6: value 470 -> 1000
Other:
- note added: "C1532"
- note added: "C16772"
Changed lines of the file:
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@@
     (stroke (width 0) (type default))
   )
+  (text "C1532" (at 132.08 99.06 0)
+    (effects (font (size 1.27 1.27)) (justify left bottom))
+  )
   (text "LOAD CELL" (at 82.55 113.665 0)
     (effects (font (size 1.27 1.27)) (justify left bottom))
   )
+  (text "C1532" (at 132.08 80.01 0)
+    (effects (font (size 1.27 1.27)) (justify left bottom))
+  )
+  (text "C16772" (at 146.05 92.71 0)
+    (effects (font (size 1.27 1.27)) (justify left bottom))
+  )
   (text "ADC" (at 130.81 113.03 0)
     (effects (font (size 1.27 1.27)) (justify left bottom))
@@
       (effects (font (size 1.27 1.27)))
     )
-    (property "Value" "470" (at 118.11 99.06 90)
+    (property "Value" "1000" (at 118.11 99.06 90)
       (effects (font (size 1.27 1.27)))
     )
@@
       (effects (font (size 1.27 1.27)))
     )
-    (property "Value" "470" (at 118.11 72.39 90)
+    (property "Value" "1000" (at 118.11 72.39 90)
       (effects (font (size 1.27 1.27)))
     )
@@
   )
   (symbol (lib_id "Device:C") (at 128.27 93.98 0) (unit 1)
-    (in_bom yes) (on_board yes) (dnp no) (fields_autoplaced)
+    (in_bom yes) (on_board yes) (dnp no)
     (property "Reference" "C2" (at 132.08 93.345 0)
       (effects (font (size 1.27 1.27)) (justify left))
     )
-    (property "Value" "47n" (at 132.08 95.885 0)
+    (property "Value" "22n" (at 132.08 95.885 0)
       (effects (font (size 1.27 1.27)) (justify left))
     )
@@
       (effects (font (size 1.27 1.27)) (justify left))
     )
-    (property "Value" "47n" (at 132.08 84.455 0)
+    (property "Value" "22n" (at 132.08 84.455 0)
       (effects (font (size 1.27 1.27)) (justify left))
     )
@@
       (effects (font (size 1.27 1.27)) (justify left))
     )
-    (property "Value" "470n" (at 146.05 89.535 0)
-      (effects (font (size 1.27 1.27)) (justify left))
-    )
+    (property "Value" "220n" (at 146.05 89.535 0)
+      (effects (font (size 1.27 1.27)) (justify left))
+    )
