File: hookup_board/kicad/hookup_board.kicad_sch (KiCad schematic)
At the start: 3 parts, among them J1 pcie_98, J2 Conn_02x25_Odd_Even, J3 Conn_02x25_Odd_Even

Commit message: Add more progress on the hookup board's layout.
Parts:
- J1: footprint common:PCIE_98_CARD -> hookup_board:PCIE_98_MINI_CARD
- J2, J3: footprint hookup_board:PinHeader_2x25_P2.00mm_Vertical_SMD -> hookup_board:PinHeader_2x25_P2.54mm_Vertical
Changed lines of the file:
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@@
       (effects (font (size 1.27 1.27)))
     )
-    (property "Footprint" "common:PCIE_98_CARD" (at 99.949 32.766 0)
+    (property "Footprint" "hookup_board:PCIE_98_MINI_CARD" (at 99.949 32.766 0)
       (effects (font (size 1.27 1.27)) hide)
     )
@@
       (effects (font (size 1.27 1.27)))
     )
-    (property "Footprint" "hookup_board:PinHeader_2x25_P2.00mm_Vertical_SMD" (at 182.88 73.66 0)
+    (property "Footprint" "hookup_board:PinHeader_2x25_P2.54mm_Vertical" (at 182.88 73.66 0)
       (effects (font (size 1.27 1.27)) hide)
     )
@@
       (effects (font (size 1.27 1.27)))
     )
-    (property "Footprint" "hookup_board:PinHeader_2x25_P2.00mm_Vertical_SMD" (at 139.7 73.66 0)
+    (property "Footprint" "hookup_board:PinHeader_2x25_P2.54mm_Vertical" (at 139.7 73.66 0)
       (effects (font (size 1.27 1.27)) hide)
     )
