File: backplane/kicad/backplane.kicad_pcb (KiCad board)
At the start: 4 copper layers, 140 x 67 mm, 14 parts, among them J1 Conn_01x02_Pin

Commit message: Cleaned up TODOs for next version of backplane.
Parts:
- added TP1: TestPoint, common:Test_Pad, F.Cu at (85.0, 94.0)
- added TP2: TestPoint, common:Test_Pad, F.Cu at (85.0, 99.1)
- added TP3: TestPoint, common:Test_Pad, F.Cu at (85.0, 88.9)
- added TP4: TestPoint, common:Test_Pad, F.Cu at (84.9, 83.8)
- J1: footprint backplane:JST_XH_B2B-XH-AM_1x02_P2.50mm_Vertical -> backplane:TerminalBlock_3P_7.62mm
- moved J1 1.39 mm to (85.3, 118.6)
Connections:
- H1 pad 1: (no net) -> unconnected-(H1-Pad1)
- H2 pad 1: (no net) -> unconnected-(H2-Pad1)
- H3 pad 1: (no net) -> unconnected-(H3-Pad1)
- H4 pad 1: (no net) -> unconnected-(H4-Pad1)
- H5 pad 1: (no net) -> unconnected-(H5-Pad1)
- H6 pad 1: (no net) -> unconnected-(H6-Pad1)
- J1 pad 1: /VIN- -> /GND
- J1 pad 2: /VIN+ -> /VIN-
Routing:
- net /VIN+: track 0.00 -> 35.2 mm
- net /VIN-: track 0.00 -> 24.4 mm
- net /+5V: track 0.00 -> 13.6 mm
Other:
- board text added: "+5V"
- board text added: "Backplane Version 0.2"
- board text added: "GND"
- board text added: "VIN+"
- board text added: "VIN-"
- board text removed: "Backplane Version 0.1"
